Commit message: minor, use config of husky from feb 2018

File: husky_ori/urdf/husky_multisense.urdf.xacro (robot description, xacro)
@@ -79,5 +79,6 @@
    <!-- Multisense -->
     <joint name="head_joint" type="fixed">
-      <origin xyz="0.315 0.0 0.593"/>
+      <!-- same as real robot in feb 2018: 31degrees-->
+      <origin xyz="0.465 0.000 0.558" rpy="0.0 0.5411 0.0" />
       <parent link="base_link" />
 <!--      <parent link="ptu_mount_link" /> -->

Commit message: compatiblity between sim and real in rvis

File: husky_ori/urdf/husky_multisense.urdf.xacro (robot description, xacro)
@@ -30,4 +30,7 @@
   <xacro:arg name="robot_namespace" default="/" />
   <xacro:arg name="urdf_extras" default="empty.urdf" />
+  <!-- real or sim - loads a different urdf  -->
+  <xacro:arg name="multisense_sim" default="false" />
+  <xacro:arg name="multisense_real" default="false" />
   <!-- Included URDF/XACRO Files -->
   <xacro:include filename="$(find husky_description)/urdf/decorations.urdf.xacro" />
@@ -36,5 +39,26 @@
   <xacro:include filename="$(find husky_description)/urdf/accessories/sick_lms1xx_mount.urdf.xacro"/>
   <xacro:include filename="$(find husky_description)/urdf/accessories/sensor_arch.urdf.xacro"/>
-  <xacro:include filename="$(find multisense_sl)/multisense_sl_sim.urdf" />
+  <xacro:if value="$(arg multisense_sim)">
+    <xacro:include filename="$(find multisense_sl)/multisense_sl_sim.urdf" />
+    <multisense name="multisense"/>
+    <!-- Multisense -->
+    <!-- same as real robot in feb 2018: 31degrees-->
+    <joint name="multisense/head_joint" type="fixed">
+      <origin xyz="0.465 0.000 0.558" rpy="0.0 0.5411 0.0" />
+      <parent link="base_link" />
+      <child link="multisense/head" />
+    </joint>
+  </xacro:if>
+  <xacro:if value="$(arg multisense_real)">
+    <xacro:include filename="$(find multisense_description)/urdf/multisenseSL/multisenseSL.urdf.xacro" />
+    <multisenseSL name="multisense" />
+    <!-- Multisense -->
+    <!-- same as real robot in feb 2018: 31degrees-->
+    <joint name="multisense/head_joint" type="fixed">
+      <origin xyz="0.465 0.000 0.558" rpy="0.0 0.5411 0.0" />
+      <parent link="base_link" />
+      <child link="multisense/head" />
+    </joint>
+  </xacro:if>
   <xacro:property name="M_PI" value="3.14159"/>
   <!-- Base Size -->
@@ -77,12 +101,4 @@
     <child link="base_footprint" />
   </joint>
-   <!-- Multisense -->
-    <joint name="head_joint" type="fixed">
-      <!-- same as real robot in feb 2018: 31degrees-->
-      <origin xyz="0.465 0.000 0.558" rpy="0.0 0.5411 0.0" />
-      <parent link="base_link" />
-<!--      <parent link="ptu_mount_link" /> -->
-      <child link="head_root" />
-    </joint>
   <!-- Interial link stores the robot's inertial information -->
   <link name="inertial_link">

Commit message: use the pitch angle of the husky as of feb 2018

File: husky_ori/urdf/husky_multisense.urdf.xacro (robot description, xacro)
@@ -56,5 +56,5 @@
     <!-- same as real robot in feb 2018: 31degrees-->
     <joint name="multisense/head_joint" type="fixed">
-      <origin xyz="0.465 0.000 0.558" rpy="0.0 0.5411 0.0" />
+      <origin xyz="0.465 0.000 0.558" rpy="0.0 0.28278 0.0" />
       <parent link="base_link" />
       <child link="multisense/head" />
