Commit message: adding basic husky with stereo for bruno

File: husky_drs/urdf/husky_multisense.urdf.xacro (robot description, xacro)
@@ -33,4 +33,5 @@
   <xacro:arg name="multisense_sim" default="false" />
   <xacro:arg name="multisense_real" default="false" />
+  <xacro:arg name="multisense_stereo" default="false" />
   <!-- Included URDF/XACRO Files -->
   <xacro:include filename="$(find husky_description)/urdf/decorations.urdf.xacro" />
@@ -39,9 +40,9 @@
   <xacro:include filename="$(find husky_description)/urdf/accessories/sick_lms1xx_mount.urdf.xacro"/>
   <xacro:include filename="$(find husky_description)/urdf/accessories/sensor_arch.urdf.xacro"/>
+  <!-- Multisense -->
+  <!-- same pitch as real robot in feb 2018: 31degrees-->
   <xacro:if value="$(arg multisense_sim)">
     <xacro:include filename="$(find multisense_sl)/multisense_sl_sim.urdf" />
     <multisense name="multisense"/>
-    <!-- Multisense -->
-    <!-- same as real robot in feb 2018: 31degrees-->
     <joint name="multisense/head_joint" type="fixed">
       <origin xyz="0.465 0.000 0.558" rpy="0.0 0.5411 0.0" />
@@ -53,8 +54,15 @@
     <xacro:include filename="$(find multisense_description)/urdf/multisenseSL/multisenseSL.urdf.xacro" />
     <multisenseSL name="multisense" />
-    <!-- Multisense -->
-    <!-- same as real robot in feb 2018: 31degrees-->
     <joint name="multisense/head_joint" type="fixed">
       <origin xyz="0.465 0.000 0.558" rpy="0.0 0.28278 0.0" />
+      <parent link="base_link" />
+      <child link="multisense/head" />
+    </joint>
+  </xacro:if>
+  <xacro:if value="$(arg multisense_stereo)">
+    <xacro:include filename="$(find husky_drs)/cameras/multisense/multisense_sl_sim_minimal_stereo.urdf" />
+    <multisense name="multisense"/>
+    <joint name="multisense/head_joint" type="fixed">
+      <origin xyz="0.465 0.000 0.558" rpy="0.0 0.5411 0.0" />
       <parent link="base_link" />
       <child link="multisense/head" />
